File: STM32 PCB Eagle/untitled.brd (EAGLE design)
At the start: 48.2 x 58.1 mm, 17 parts, among them IC1 LTV-846S, U1 SN65HVD230/1

Commit message: Added serial debug hdr and minor rerouting
Parts:
- added H1: 1X2, headers(.1in):1X2
- moved R9 4.49 mm to (40.0, 54.0)
- moved R3 0.28 mm to (25.3, 16.3)
- turned PSU1 to 0 degrees
Connections:
- new net RX1: H1.2, STM32.P$27
- new net TX1: H1.1, STM32.P$26
Routing:
- net TX1: track 0.00 -> 8.87 mm
- net RX1: track 0.00 -> 8.87 mm
- net PB11: track 61.9 -> 69.3 mm
- net GND: track 32.6 -> 27.2 mm
- net N$9: track 3.44 -> 7.57 mm
- net 12V: track 12.2 -> 15.7 mm
- net 3V3: track 11.9 -> 9.45 mm
- net PB14: track 43.5 -> 44.2 mm
Other:
- board text added: "T4R Auto-Headlights v1"
- board text added: "TX1 RX1"
- board text added: "github.com/ColtB45/T4R-Auto-Headlights"
- board text removed: "T4R Auto-Lights v1"

Commit message: Alterations to keep MPX resistance below 200 ohms
The MPX only allows a resistance of < 250 ohms. I've made the following alterations to keep the LTV-846 resistance to MPX ~200 ohms. The resistors between the LTV-846 and the MPX were there only to reduce current through the LTV. In conditions I've observed, the LTV-846 should be under it's maximum ratings without the resistors. If the current draw through the LTV-846 spikes for some reason, there is no risk to the MPX or STM32.
Removing these resistors should have no detrimental impact.
Parts:
- removed R6, R9: 47k ohm, rcl:R1206
- removed R7, R8: 1k ohm, rcl:R1206
- R1, R3, R4: value 1k ohm -> 47 ohm
- R5: value 1k ohm -> 47k ohm
- moved R5 31.2 mm to (40.0, 54.0), turned to 180 degrees
Connections:
- removed net N$1: IC1.16, R5.1
- removed net N$3: IC1.13, R6.1
- removed net N$5: IC1.12, R7.1
- removed net N$7: IC1.10, R8.1
- net DRL_MPX: now also IC1.12; no longer R7.2
- net HDL_MPX: now also IC1.16; no longer R5.2
- net N$9: now also R5.2; no longer R9.2
- net PB11: now also R5.1; no longer R9.1
- net PB14: now also IC1.13; no longer R6.2
- net TL_MPX: now also IC1.10; no longer R8.2
Routing:
- net HDL_MPX: track 4.25 -> 33.5 mm
- net N$1: track 26.6 -> 0.00 mm
- net N$5: track 20.6 -> 0.00 mm
- net DRL_MPX: track 4.03 -> 21.3 mm
- net TL_MPX: track 4.47 -> 13.1 mm
- net N$7: track 7.28 -> 0.00 mm
- net GND: track 27.2 -> 21.7 mm, vias 8 -> 7
- net N$3: track 4.44 -> 0.00 mm
- net CANL: track 46.0 -> 50.0 mm
- net CANH: track 49.0 -> 51.1 mm
- net PB14: track 44.2 -> 46.3 mm
- net 12V: track 15.7 -> 16.2 mm

Commit message: This is the version sent to printing.
Parts:
- H1: value 1X2 -> 1X3; device headers(.1in):1X2 -> headers(.1in):1X3
- moved PSU1 7.11 mm to (30.7, 10.5), turned to 180 degrees
- moved C3 5.61 mm to (31.8, 5.97)
- moved C2 5.43 mm to (25.9, 5.97), turned to 0 degrees
- moved R5 3.91 mm to (36.8, 51.7)
- moved IC1 3.86 mm to (33.7, 34.3)
- moved R4 3.86 mm to (24.8, 26.7)
- moved R1 3.74 mm to (24.8, 39.5)
- moved H1 2.81 mm to (28.8, 16.4)
- moved R2 2.79 mm to (35.7, 16.4)
- moved C1 2.30 mm to (37.8, 8.64), turned to 270 degrees
- moved U1 2.29 mm to (28.1, 49.8)
- moved R3 2.17 mm to (24.5, 14.2)
- moved U$1 1.59 mm to (42.4, 15.1)
Connections:
- new net PA1: R5.1, STM32.P$6
- net 12V: now also U$1.2; no longer U$1.1
- net CANH: now also U$1.7; no longer U$1.3
- net CANL: now also U$1.8; no longer U$1.4
- net GND: now also H1.3, U$1.1; no longer U$1.2
- net HDL_MPX: now also U$1.3; no longer U$1.7
- net PB11: no longer R5.1
- net TL_MPX: now also U$1.4; no longer U$1.8
Routing:
- net PB11: track 69.3 -> 0.00 mm
- net PA1: track 0.00 -> 39.3 mm
- net CANL: track 50.0 -> 36.4 mm
- net CANH: track 51.1 -> 39.0 mm
- net PB14: track 46.3 -> 40.9 mm
- net TL_MPX: track 13.1 -> 18.4 mm, vias 0 -> 1
- net DRL_MPX: track 21.3 -> 17.2 mm
- net 3V3: track 9.45 -> 12.9 mm, vias 4 -> 3
- net GND: track 21.7 -> 18.4 mm, vias 7 -> 1
- net N$9: track 7.57 -> 4.27 mm
- net N$4: track 24.6 -> 22.2 mm
- net PA11: track 8.36 -> 6.15 mm
- net 12V: track 16.2 -> 14.1 mm
- net PB15: track 33.2 -> 31.1 mm
- net N$6: track 22.6 -> 24.5 mm
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Other:
- board size 48.2 x 58.1 mm -> 45.7 x 53.3 mm
- board text added: "Magic smoke containment device"
- board text added: "TX RX GND"
- board text removed: "Change magic smoke every 1337 days"
- board text removed: "T4R Auto-Headlights v1"
- board text removed: "TX1 RX1"
